File: Sixty-n8k/Sixty-n8k.kicad_pcb (KiCad board)
At the start: 4 copper layers, 149.9 x 99.7 mm, 69 parts, among them J1 USB4085-GF-A_REVB, J2 SD_CARD_PORT, J3 Conn_02x32_Odd_Even, J4 Conn_01x02, SW1 RESET, SW2 DEBUG, U1 74LS05, U10 74HC164, U11 74LS393, U12 22V10C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

Commit message: Fixes a couple of small issues
Parts:
- J4: value Conn_01x02 -> Conn_01x03_Pin; footprint Connector_PinHeader_2.54mm:PinHeader_1x02_P2.54mm_Vertical -> Connector_PinHeader_2.54mm:PinHeader_1x03_P2.54mm_Vertical
- moved J4 34.9 mm to (190.4, 117.4), turned to -90 degrees
Connections:
- J4 pad 1: ~{AS} -> +5V
- J4 pad 2: BERR_WATCHDOG -> Net-(J4-Pin_2)
- RN2 pad 2: BERR_WATCHDOG -> unconnected-(RN2-R1-Pad2)
- RN2 pad 4: ~{HALT} -> ~{RES}
- RN2 pad 5: HALT -> ~{HALT}
- RN2 pad 6: ~{RES} -> HALT
- U11 pad 1: E -> Net-(J4-Pin_2)
- U11 pad 2: BERR_WATCHDOG -> ~{AS}
Routing:
- net BERR_WATCHDOG: track 37.1 -> 0.00 mm
- net Net-(J4-Pin_2): track 0.00 -> 30.2 mm
- net E: track 119.8 -> 146.0 mm, vias 3 -> 4
- net ~{AS}: track 179.5 -> 203.8 mm, vias 0 -> 1
- net HALT: track 23.0 -> 35.7 mm
- net ~{CS_ROM}_{ODD}: track 158.1 -> 161.3 mm
- net CLK_{CPU}: track 178.9 -> 179.9 mm
Other:
- board text added: "Watchdog"
- board text removed: "Watchdog?"

Commit message: PCB cleanup
Routing:
- net ~{VMA}: track 92.3 -> 56.7 mm, vias 8 -> 2
Other:
- board text added: "+5V"
- board text added: "CS"
- board text added: "Disabled"
- board text added: "MISO"
- board text added: "MOSI"

Commit message: footprint fix :(
Parts:
- removed G1: LOGO, graphics:Shaka
- removed G2: LOGO, graphics:MadeInAMS
- U6: footprint Package_DIP:DIP-64_W25.4mm_Socket -> Package_DIP:DIP-64_W22.86mm_Socket
