File: Sixty-n8k/Sixty-n8k.kicad_pcb (KiCad board)
At the start: 4 copper layers, 149.9 x 99.7 mm, 67 parts, among them J1 USB4085-GF-A_REVB, J2 SD_CARD_PORT, J3 Conn_02x32_Odd_Even, J4 Conn_01x03_Pin, SW1 RESET, SW2 DEBUG, U1 74LS05, U10 74HC164, U11 74LS393, U12 22V10C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

Commit message: Open collector via schottky diode for NMI
Parts:
- added D5: D_Schottky, Diode_THT:D_DO-41_SOD81_P7.62mm_Horizontal, F.Cu at (111.5, 101.4)
- D2: value HALT -> RUNNING
Connections:
- R4 pad 2: Net-(R4-Pad2) -> /RUNNING
- RN2 pad 6: HALT -> unconnected-(RN2-R5-Pad6)
- U1 pad 10: HALT -> /RUNNING
- U1 pad 8: Net-(R4-Pad2) -> unconnected-(U1-Pad8)
- U1 pad 9: HALT -> unconnected-(U1-Pad9)
- U16 pad 7: unconnected-(U16-O7-Pad7) -> Net-(D5-K)
Routing:
- net Net-(D5-K): track 0.00 -> 78.2 mm
- net Net-(R4-Pad2): track 71.9 -> 0.00 mm
- net /RUNNING: track 0.00 -> 70.0 mm
- net HALT: track 35.7 -> 0.00 mm
- net ~{VPA}: track 38.4 -> 73.6 mm, vias 0 -> 1
- net /A14: track 169.1 -> 173.9 mm
- net /A17: track 171.9 -> 173.2 mm
- net /A18: track 157.6 -> 158.7 mm
Other:
- board text added: "PWR"
- board text added: "RUN"
- board text added: "RX"
- board text added: "TX"

Commit message: Re-added logo
Parts:
- added G1: LOGO, graphics:Shaka, F.Cu at (115.5, 56.9)
- added G2: LOGO, graphics:MadeInAMS, F.Cu at (124.3, 56.8)

Commit message: Fixed short trace to CC resistor
Connections:
- U1 pad 9: unconnected-(U1-Pad9) -> GND
Routing:
- net /A14: track 173.9 -> 173.0 mm
