File: Sixty-n8k/Sixty-n8k.kicad_sch (KiCad schematic)
At the start: 67 parts, among them J1 USB4085-GF-A_REVB, J2 SD_CARD_PORT, J3 Conn_02x32_Odd_Even, J4 Conn_01x02, SW1 RESET, SW2 DEBUG, U1 74LS05, U10 74HC164, U11 74LS393, U12 22V10C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

Commit message: Formatting changes
Connections:
- net D6: no longer U4.20 (DQ6)

Commit message: Removed pullup on RWb
Connections:
- net D6: now also U4.20 (DQ6)
- net R~{W}: no longer RN3.5 (R4)
- net ~{BERR}: now also J3.40 (Pin_40); no longer J3.44 (Pin_44)
- net ~{BGACK}: now also J3.46 (Pin_46); no longer J3.60 (Pin_60)
- net ~{BG}: now also J3.42 (Pin_42); no longer J3.40 (Pin_40)
- net ~{BR}: now also J3.44 (Pin_44); no longer J3.42 (Pin_42)
Changed lines of the file:
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@@
   (no_connect (at 62.23 152.4))
   (no_connect (at 361.95 194.31))
-  (no_connect (at 58.42 327.66))
   (no_connect (at 527.05 199.39))
   (no_connect (at 336.55 327.66))
@@
   (no_connect (at 273.05 278.13))
   (no_connect (at 361.95 196.85))
+  (no_connect (at 532.13 90.17))
   (no_connect (at 438.15 294.64))
   (no_connect (at 194.31 208.28))
@@
     (stroke (width 0) (type default))
   )
-  (wire (pts (xy 529.59 90.17) (xy 532.13 90.17))
-    (stroke (width 0) (type default))
-  )
   (wire (pts (xy 323.85 48.26) (xy 328.93 48.26))
     (stroke (width 0) (type default))
@@
     (stroke (width 0) (type default))
   )
-  (wire (pts (xy 355.6 50.8) (xy 359.41 50.8))
+  (wire (pts (xy 354.33 50.8) (xy 359.41 50.8))
     (stroke (width 0) (type default))
   )
@@
     (stroke (width 0) (type default))
   )
-  (wire (pts (xy 58.42 320.04) (xy 60.96 320.04))
+  (wire (pts (xy 58.42 322.58) (xy 60.96 322.58))
     (stroke (width 0) (type default))
   )
@@
     (stroke (width 0) (type default))
   )
-  (wire (pts (xy 359.41 50.8) (xy 360.68 50.8))
-    (stroke (width 0) (type default))
-  )
   (wire (pts (xy 323.85 134.62) (xy 328.93 134.62))
     (stroke (width 0) (type default))
@@
     (stroke (width 0) (type solid))
   )
-  (wire (pts (xy 58.42 322.58) (xy 60.96 322.58))
+  (wire (pts (xy 58.42 325.12) (xy 60.96 325.12))
     (stroke (width 0) (type default))
   )
@@
     (stroke (width 0) (type default))
   )
-  (wire (pts (xy 58.42 345.44) (xy 60.96 345.44))
+  (wire (pts (xy 58.42 327.66) (xy 60.96 327.66))
     (stroke (width 0) (type default))
   )
@@
     (stroke (width 0) (type default))
   )
-  (wire (pts (xy 58.42 325.12) (xy 60.96 325.12))
+  (wire (pts (xy 58.42 320.04) (xy 60.96 320.04))
     (stroke (width 0) (type default))
   )
@@
     )
   )
-  (global_label "~{BR}" (shape output) (at 60.96 322.58 0) (fields_autoplaced)
+  (global_label "~{BR}" (shape output) (at 60.96 325.12 0) (fields_autoplaced)
     (effects (font (size 1.27 1.27)) (justify left))
-    (property "Intersheetrefs" "${INTERSHEET_REFS}" (at 66.4058 322.58 0)
+    (property "Intersheetrefs" "${INTERSHEET_REFS}" (at 66.4058 325.12 0)
       (effects (font (size 1.27 1.27)) (justify left) hide)
     )
@@
     )
   )
-  (global_label "R~{W}" (shape input) (at 529.59 90.17 180) (fields_autoplaced)
-    (effects (font (size 1.27 1.27)) (justify right))
-    (property "Intersheetrefs" "${INTERSHEET_REFS}" (at 523.9628 90.17 0)
-      (effects (font (size 1.27 1.27)) (justify right) hide)
-    )
-  )
   (global_label "~{LDS}" (shape input) (at 231.14 222.25 180) (fields_autoplaced)
     (effects (font (size 1.27 1.27)) (justify right))
@@
     )
   )
-  (global_label "~{BERR}" (shape input) (at 60.96 325.12 0) (fields_autoplaced)
+  (global_label "~{BERR}" (shape input) (at 60.96 320.04 0) (fields_autoplaced)
     (effects (font (size 1.27 1.27)) (justify left))
-    (property "Intersheetrefs" "${INTERSHEET_REFS}" (at 68.8248 325.12 0)
+    (property "Intersheetrefs" "${INTERSHEET_REFS}" (at 68.8248 320.04 0)
       (effects (font (size 1.27 1.27)) (justify left) hide)
     )
@@
     )
   )
-  (global_label "~{BG}" (shape input) (at 60.96 320.04 0) (fields_autoplaced)
+  (global_label "~{BG}" (shape input) (at 60.96 322.58 0) (fields_autoplaced)
     (effects (font (size 1.27 1.27)) (justify left))
-    (property "Intersheetrefs" "${INTERSHEET_REFS}" (at 66.4058 320.04 0)
+    (property "Intersheetrefs" "${INTERSHEET_REFS}" (at 66.4058 322.58 0)
       (effects (font (size 1.27 1.27)) (justify left) hide)
     )
@@
     )
   )
-  (global_label "~{BGACK}" (shape output) (at 60.96 345.44 0) (fields_autoplaced)
+  (global_label "~{BGACK}" (shape output) (at 60.96 327.66 0) (fields_autoplaced)
     (effects (font (size 1.27 1.27)) (justify left))
-    (property "Intersheetrefs" "${INTERSHEET_REFS}" (at 70.0344 345.44 0)
+    (property "Intersheetrefs" "${INTERSHEET_REFS}" (at 70.0344 327.66 0)
       (effects (font (size 1.27 1.27)) (justify left) hide)
     )

Commit message: Fixes a couple of small issues
Parts:
- removed J4: Conn_01x02, Connector_PinHeader_2.54mm:PinHeader_1x02_P2.54mm_Vertical, symbol Connector_Generic:Conn_01x02
- added J4: Conn_01x03_Pin, Connector_PinHeader_2.54mm:PinHeader_1x03_P2.54mm_Vertical, symbol Connector:Conn_01x03_Pin
Connections:
- net +5V: now also J4.1 (Pin_1)
- net E: now also J4.3 (Pin_3); no longer U11.1 (CP)
- net HALT: now also RN2.6 (R5); no longer RN2.5 (R4)
- net ~{AS}: now also U11.2 (MR)
- net ~{HALT}: now also RN2.5 (R4); no longer RN2.4 (R3)
- net ~{RES}: now also RN2.4 (R3); no longer RN2.6 (R5)
- net BERR_WATCHDOG: no longer names the net of RN2.2 (R1)
- net BERR_WATCHDOG: no longer U11.2 (MR)
- new net: J4.2 (Pin_2), U11.1 (CP)
- no-connect marks 54 -> 56
Changed lines of the file:
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@@
   (junction (at 184.15 370.84) (diameter 0) (color 0 0 0 0)
   )
-  (junction (at 334.01 199.39) (diameter 0) (color 0 0 0 0)
-  )
   (junction (at 359.41 127) (diameter 0) (color 0 0 0 0)
   )
@@
   (no_connect (at 44.45 203.2))
   (no_connect (at 62.23 149.86))
+  (no_connect (at 532.13 43.18))
   (no_connect (at 194.31 213.36))
+  (no_connect (at 58.42 345.44))
   (no_connect (at 438.15 309.88))
   (no_connect (at 458.47 307.34))
@@
     (stroke (width 0) (type default))
   )
-  (wire (pts (xy 529.59 43.18) (xy 532.13 43.18))
-    (stroke (width 0) (type default))
-  )
   (wire (pts (xy 171.45 203.2) (xy 173.99 203.2))
     (stroke (width 0) (type default))
@@
     (stroke (width 0) (type default))
   )
+  (wire (pts (xy 330.2 189.23) (xy 330.2 191.77))
+    (stroke (width 0) (type default))
+  )
   (wire (pts (xy 458.47 312.42) (xy 461.01 312.42))
     (stroke (width 0) (type default))
@@
     (stroke (width 0) (type default))
   )
-  (wire (pts (xy 331.47 210.82) (xy 334.01 210.82))
-    (stroke (width 0) (type default))
-  )
   (wire (pts (xy 58.42 322.58) (xy 60.96 322.58))
     (stroke (width 0) (type default))
@@
     (stroke (width 0) (type default))
   )
-  (wire (pts (xy 529.59 48.26) (xy 532.13 48.26))
+  (wire (pts (xy 529.59 50.8) (xy 532.13 50.8))
     (stroke (width 0) (type default))
   )
@@
     (stroke (width 0) (type default))
   )
-  (wire (pts (xy 326.39 199.39) (xy 334.01 199.39))
+  (wire (pts (xy 334.01 199.39) (xy 336.55 199.39))
     (stroke (width 0) (type default))
   )
@@
     (stroke (width 0) (type default))
   )
-  (wire (pts (xy 320.04 199.39) (xy 323.85 199.39))
-    (stroke (width 0) (type default))
-  )
   (wire (pts (xy 213.36 58.42) (xy 215.9 58.42))
     (stroke (width 0) (type default))
@@
     (stroke (width 0) (type default))
   )
-  (wire (pts (xy 529.59 53.34) (xy 532.13 53.34))
+  (wire (pts (xy 529.59 48.26) (xy 532.13 48.26))
     (stroke (width 0) (type default))
   )
@@
     (stroke (width 0) (type default))
   )
-  (wire (pts (xy 334.01 199.39) (xy 336.55 199.39))
-    (stroke (width 0) (type default))
-  )
   (wire (pts (xy 63.5 274.32) (xy 58.42 274.32))
     (stroke (width 0) (type default))
@@
     (stroke (width 0) (type default))
   )
-  (wire (pts (xy 334.01 191.77) (xy 336.55 191.77))
+  (wire (pts (xy 325.12 189.23) (xy 327.66 189.23))
     (stroke (width 0) (type default))
   )
@@
     (stroke (width 0) (type default))
   )
+  (wire (pts (xy 330.2 191.77) (xy 336.55 191.77))
+    (stroke (width 0) (type default))
+  )
   (bus (pts (xy 274.32 45.72) (xy 274.32 48.26))
     (stroke (width 0) (type default))
@@
     (stroke (width 0) (type default))
   )
-  (wire (pts (xy 334.01 210.82) (xy 334.01 199.39))
-    (stroke (width 0) (type default))
-  )
   (bus (pts (xy 66.04 289.56) (xy 66.04 287.02))
     (stroke (width 0) (type default))
@@
     (stroke (width 0) (type default))
   )
+  (wire (pts (xy 332.74 189.23) (xy 336.55 189.23))
+    (stroke (width 0) (type default))
+  )
   (wire (pts (xy 410.21 48.26) (xy 417.83 48.26))
     (stroke (width 0) (type default))
@@
     (stroke (width 0) (type default))
   )
-  (wire (pts (xy 529.59 50.8) (xy 532.13 50.8))
+  (wire (pts (xy 529.59 53.34) (xy 532.13 53.34))
     (stroke (width 0) (type default))
   )
@@
     )
   )
-  (global_label "HALT" (shape input) (at 529.59 50.8 180) (fields_autoplaced)
+  (global_label "HALT" (shape input) (at 529.59 53.34 180) (fields_autoplaced)
     (effects (font (size 1.27 1.27)) (justify right))
-    (property "Intersheetrefs" "${INTERSHEET_REFS}" (at 522.2694 50.8 0)
+    (property "Intersheetrefs" "${INTERSHEET_REFS}" (at 522.2694 53.34 0)
       (effects (font (size 1.27 1.27)) (justify right) hide)
     )
@@
     )
   )
-  (global_label "BERR_WATCHDOG" (shape input) (at 331.47 210.82 180) (fields_autoplaced)
-    (effects (font (size 1.27 1.27)) (justify right))
-    (property "Intersheetrefs" "${INTERSHEET_REFS}" (at 312.659 210.82 0)
-      (effects (font (size 1.27 1.27)) (justify right) hide)
-    )
-  )
   (global_label "~{BGACK}" (shape input) (at 213.36 53.34 180) (fields_autoplaced)
     (effects (font (size 1.27 1.27)) (justify right))
@@
     )
   )
-  (global_label "~{HALT}" (shape input) (at 529.59 48.26 180) (fields_autoplaced)
+  (global_label "~{HALT}" (shape input) (at 529.59 50.8 180) (fields_autoplaced)
     (effects (font (size 1.27 1.27)) (justify right))
-    (property "Intersheetrefs" "${INTERSHEET_REFS}" (at 522.2694 48.26 0)
+    (property "Intersheetrefs" "${INTERSHEET_REFS}" (at 522.2694 50.8 0)
       (effects (font (size 1.27 1.27)) (justify right) hide)
     )
@@
     )
   )
-  (global_label "BERR_WATCHDOG" (shape input) (at 529.59 43.18 180) (fields_autoplaced)
-    (effects (font (size 1.27 1.27)) (justify right))
-    (property "Intersheetrefs" "${INTERSHEET_REFS}" (at 510.779 43.18 0)
-      (effects (font (size 1.27 1.27)) (justify right) hide)
-    )
-  )
   (global_label "~{AS}" (shape input) (at 529.59 82.55 180) (fields_autoplaced)
     (effects (font (size 1.27 1.27)) (justify right))
@@
     )
   )
-  (global_label "E" (shape input) (at 334.01 191.77 180) (fields_autoplaced)
+  (global_label "E" (shape input) (at 325.12 189.23 180) (fields_autoplaced)
     (effects (font (size 1.27 1.27)) (justify right))
-    (property "Intersheetrefs" "${INTERSHEET_REFS}" (at 329.9552 191.77 0)
+    (property "Intersheetrefs" "${INTERSHEET_REFS}" (at 321.0652 189.23 0)
       (effects (font (size 1.27 1.27)) (justify right) hide)
     )
@@
     )
   )
-  (global_label "~{RES}" (shape input) (at 529.59 53.34 180) (fields_autoplaced)
+  (global_label "~{RES}" (shape input) (at 529.59 48.26 180) (fields_autoplaced)
     (effects (font (size 1.27 1.27)) (justify right))
-    (property "Intersheetrefs" "${INTERSHEET_REFS}" (at 523.0557 53.34 0)
+    (property "Intersheetrefs" "${INTERSHEET_REFS}" (at 523.0557 48.26 0)
       (effects (font (size 1.27 1.27)) (justify right) hide)
     )
@@
     )
   )
-  (global_label "~{AS}" (shape input) (at 320.04 199.39 180) (fields_autoplaced)
+  (global_label "~{AS}" (shape input) (at 334.01 199.39 180) (fields_autoplaced)
     (effects (font (size 1.27 1.27)) (justify right))
-    (property "Intersheetrefs" "${INTERSHEET_REFS}" (at 314.8361 199.39 0)
+    (property "Intersheetrefs" "${INTERSHEET_REFS}" (at 328.8061 199.39 0)
       (effects (font (size 1.27 1.27)) (justify right) hide)
     )
@@
     )
   )
+  (symbol (lib_id "power:+5V") (at 336.55 189.23 0) (unit 1)
+    (in_bom yes) (on_board yes) (dnp no) (fields_autoplaced)
+    (property "Reference" "#PWR048" (at 336.55 193.04 0)
+      (effects (font (size 1.27 1.27)) hide)
+    )
+    (property "Value" "+5V" (at 336.55 184.15 0)
+      (effects (font (size 1.27 1.27)))
+    )
+    (property "Footprint" "" (at 336.55 189.23 0)
+      (effects (font (size 1.27 1.27)) hide)
+    )
+    (property "Datasheet" "" (at 336.55 189.23 0)
+      (effects (font (size 1.27 1.27)) hide)
+    )
+    (pin "1")
+    (instances
+      (project "Sixty-n8k"
+        (path "/899701f7-f496-45c9-a35e-7f376afd1eaf"
+          (reference "#PWR048") (unit 1)
+        )
+      )
+    )
+  )
   (symbol (lib_id "power:+5V") (at 341.63 29.21 0) (unit 1)
     (in_bom yes) (on_board yes) (dnp no) (fields_autoplaced)
@@
     )
   )
-  (symbol (lib_id "Connector_Generic:Conn_01x02") (at 323.85 204.47 90) (mirror x) (unit 1)
+  (symbol (lib_id "Connector:Conn_01x03_Pin") (at 330.2 184.15 270) (unit 1)
     (in_bom yes) (on_board yes) (dnp no)
-    (property "Reference" "J4" (at 321.31 203.2 90)
-      (effects (font (size 1.27 1.27)) (justify left))
+    (property "Reference" "J4" (at 330.2 179.07 90)
+      (effects (font (size 1.27 1.27)))
     )
-    (property "Value" "Conn_01x02" (at 321.31 205.74 90)
-      (effects (font (size 1.27 1.27)) (justify left))
+    (property "Value" "Conn_01x03_Pin" (at 318.77 185.42 90)
+      (effects (font (size 1.27 1.27)))
     )
-    (property "Footprint" "Connector_PinHeader_2.54mm:PinHeader_1x02_P2.54mm_Vertical" (at 323.85 204.47 0)
+    (property "Footprint" "Connector_PinHeader_2.54mm:PinHeader_1x03_P2.54mm_Vertical" (at 330.2 184.15 0)
       (effects (font (size 1.27 1.27)) hide)
     )
-    (property "Datasheet" "~" (at 323.85 204.47 0)
+    (property "Datasheet" "~" (at 330.2 184.15 0)
       (effects (font (size 1.27 1.27)) hide)
     )
-    (pin "1")
     (pin "2")
+    (pin "3")
+    (pin "1")
     (instances
       (project "Sixty-n8k"

Commit message: footprint fix :(
Parts:
- D2: value HALT -> RUNNING
- U6: footprint Package_DIP:DIP-64_W25.4mm_Socket -> Package_DIP:DIP-64_W22.86mm_Socket
Connections:
- net at U1.8: no longer R4.2
- net HALT renamed RUNNING
- net RUNNING: now also R4.2; no longer U1.9
Other:
- moved on the sheet: D2, R4
Changed lines of the file:
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@@
     (stroke (width 0) (type default))
   )
-  (wire (pts (xy 123.19 88.9) (xy 123.19 91.44))
+  (wire (pts (xy 107.95 88.9) (xy 107.95 91.44))
     (stroke (width 0) (type default))
   )
@@
     (stroke (width 0) (type default))
   )
-  (wire (pts (xy 102.87 91.44) (xy 105.41 91.44))
-    (stroke (width 0) (type default))
-  )
   (wire (pts (xy 266.7 142.24) (xy 271.78 142.24))
     (stroke (width 0) (type default))
@@
     (stroke (width 0) (type default))
   )
-  (wire (pts (xy 115.57 91.44) (xy 113.03 91.44))
+  (wire (pts (xy 100.33 91.44) (xy 97.79 91.44))
     (stroke (width 0) (type default))
   )
@@
     (stroke (width 0) (type default))
   )
-  (wire (pts (xy 82.55 91.44) (xy 87.63 91.44))
+  (wire (pts (xy 82.55 91.44) (xy 90.17 91.44))
     (stroke (width 0) (type default))
   )
@@
     (effects (font (size 1.27 1.27)) (justify left bottom))
   )
-  (label "HALT" (at 82.55 91.44 0) (fields_autoplaced)
+  (label "RUNNING" (at 82.55 91.44 0) (fields_autoplaced)
     (effects (font (size 1.27 1.27)) (justify left bottom))
   )
@@
     )
   )
-  (global_label "HALT" (shape input) (at 529.59 53.34 180) (fields_autoplaced)
+  (global_label "RUNNING" (shape input) (at 529.59 53.34 180) (fields_autoplaced)
     (effects (font (size 1.27 1.27)) (justify right))
-    (property "Intersheetrefs" "${INTERSHEET_REFS}" (at 522.2694 53.34 0)
+    (property "Intersheetrefs" "${INTERSHEET_REFS}" (at 518.2174 53.34 0)
       (effects (font (size 1.27 1.27)) (justify right) hide)
     )
@@
     )
   )
-  (symbol (lib_id "Device:R") (at 109.22 91.44 270) (unit 1)
+  (symbol (lib_id "Device:R") (at 93.98 91.44 270) (unit 1)
     (in_bom yes) (on_board yes) (dnp no)
-    (property "Reference" "R4" (at 109.22 88.9 90)
+    (property "Reference" "R4" (at 93.98 88.9 90)
       (effects (font (size 1.27 1.27)))
     )
-    (property "Value" "330" (at 109.22 91.44 90)
+    (property "Value" "330" (at 93.98 91.44 90)
       (effects (font (size 1.27 1.27)))
     )
-    (property "Footprint" "Resistor_THT:R_Axial_DIN0207_L6.3mm_D2.5mm_P7.62mm_Horizontal" (at 109.22 91.44 0)
+    (property "Footprint" "Resistor_THT:R_Axial_DIN0207_L6.3mm_D2.5mm_P7.62mm_Horizontal" (at 93.98 91.44 0)
       (effects (font (size 1.27 1.27)) hide)
     )
-    (property "Datasheet" "~" (at 109.22 91.44 0)
+    (property "Datasheet" "~" (at 93.98 91.44 0)
       (effects (font (size 1.27 1.27)) hide)
     )
@@
     )
   )
+  (symbol (lib_id "74xx:74LS05") (at 172.72 85.725 0) (unit 4)
+    (in_bom yes) (on_board yes) (dnp no) (fields_autoplaced)
+    (property "Reference" "U1" (at 172.72 77.597 0)
+      (effects (font (size 1.27 1.27)))
+    )
+    (property "Value" "74LS05" (at 172.72 80.137 0)
+      (effects (font (size 1.27 1.27)))
+    )
+    (property "Footprint" "Package_DIP:DIP-14_W7.62mm_Socket" (at 172.72 85.725 0)
+      (effects (font (size 1.27 1.27)) hide)
+    )
+    (property "Datasheet" "http://www.ti.com/lit/gpn/sn74LS05" (at 172.72 85.725 0)
+      (effects (font (size 1.27 1.27)) hide)
+    )
+    (pin "1")
+    (pin "2")
+    (pin "3")
+    (pin "4")
+    (pin "5")
+    (pin "6")
+    (pin "8")
+    (pin "9")
+    (pin "10")
+    (pin "11")
+    (pin "12")
+    (pin "13")
+    (pin "14")
+    (pin "7")
+    (instances
+      (project "Sixty-n8k"
+        (path "/899701f7-f496-45c9-a35e-7f376afd1eaf"
+          (reference "U1") (unit 4)
+        )
+      )
+    )
+  )
   (symbol (lib_id "power:+5V") (at 52.07 193.04 0) (unit 1)
     (in_bom yes) (on_board yes) (dnp no) (fields_autoplaced)
@@
       (effects (font (size 1.27 1.27)) (justify left))
     )
-    (property "Footprint" "Package_DIP:DIP-64_W25.4mm_Socket" (at 241.3 91.44 0)
+    (property "Footprint" "Package_DIP:DIP-64_W22.86mm_Socket" (at 241.3 91.44 0)
       (effects (font (size 1.27 1.27)) hide)
     )
@@
     )
   )
-  (symbol (lib_id "power:+5V") (at 123.19 88.9 0) (unit 1)
+  (symbol (lib_id "power:+5V") (at 107.95 88.9 0) (unit 1)
     (in_bom yes) (on_board yes) (dnp no) (fields_autoplaced)
-    (property "Reference" "#PWR018" (at 123.19 92.71 0)
+    (property "Reference" "#PWR018" (at 107.95 92.71 0)
       (effects (font (size 1.27 1.27)) hide)
     )
-    (property "Value" "+5V" (at 123.19 83.82 0)
+    (property "Value" "+5V" (at 107.95 83.82 0)
       (effects (font (size 1.27 1.27)))
     )
-    (property "Footprint" "" (at 123.19 88.9 0)
+    (property "Footprint" "" (at 107.95 88.9 0)
       (effects (font (size 1.27 1.27)) hide)
     )
-    (property "Datasheet" "" (at 123.19 88.9 0)
+    (property "Datasheet" "" (at 107.95 88.9 0)
       (effects (font (size 1.27 1.27)) hide)
     )
@@
     )
   )
-  (symbol (lib_id "Device:LED") (at 119.38 91.44 0) (unit 1)
+  (symbol (lib_id "Device:LED") (at 104.14 91.44 0) (unit 1)
     (in_bom yes) (on_board yes) (dnp no)
-    (property "Reference" "D2" (at 119.2022 85.9282 0)
+    (property "Reference" "D2" (at 103.9622 85.9282 0)
       (effects (font (size 1.27 1.27)))
     )
-    (property "Value" "HALT" (at 119.2022 88.2396 0)
+    (property "Value" "RUNNING" (at 103.9622 88.2396 0)
       (effects (font (size 1.27 1.27)))
     )
-    (property "Footprint" "LED_THT:LED_D3.0mm" (at 119.38 91.44 0)
+    (property "Footprint" "LED_THT:LED_D3.0mm" (at 104.14 91.44 0)
       (effects (font (size 1.27 1.27)) hide)
     )
-    (property "Datasheet" "~" (at 119.38 91.44 0)
+    (property "Datasheet" "~" (at 104.14 91.44 0)
       (effects (font (size 1.27 1.27)) hide)
     )
@@
     )
   )
-  (symbol (lib_id "74xx:74LS05") (at 95.25 91.44 0) (unit 4)
-    (in_bom yes) (on_board yes) (dnp no) (fields_autoplaced)
-    (property "Reference" "U1" (at 95.25 83.312 0)
-      (effects (font (size 1.27 1.27)))
-    )
-    (property "Value" "74LS05" (at 95.25 85.852 0)
-      (effects (font (size 1.27 1.27)))
-    )
-    (property "Footprint" "Package_DIP:DIP-14_W7.62mm_Socket" (at 95.25 91.44 0)
-      (effects (font (size 1.27 1.27)) hide)
-    )
-    (property "Datasheet" "http://www.ti.com/lit/gpn/sn74LS05" (at 95.25 91.44 0)
-      (effects (font (size 1.27 1.27)) hide)
-    )
-    (pin "1")
-    (pin "2")
-    (pin "3")
-    (pin "4")
-    (pin "5")
-    (pin "6")
-    (pin "8")
-    (pin "9")
-    (pin "10")
-    (pin "11")
-    (pin "12")
-    (pin "13")
-    (pin "14")
-    (pin "7")
-    (instances
-      (project "Sixty-n8k"
-        (path "/899701f7-f496-45c9-a35e-7f376afd1eaf"
-          (reference "U1") (unit 4)
-        )
-      )
-    )
-  )
   (symbol (lib_id "Device:C_Small") (at 293.37 383.54 0) (unit 1)
     (in_bom yes) (on_board yes) (dnp no) (fields_autoplaced)
@@
       (effects (font (size 1.27 1.27)) hide)
     )
+    (pin "1")
     (pin "2")
     (pin "3")
-    (pin "1")
     (instances
       (project "Sixty-n8k"
