File: Sixty-n8k/Sixty-n8k.kicad_sch (KiCad schematic)
At the start: 68 parts, among them J1 USB4085-GF-A_REVB, J2 SD_CARD_PORT, J3 Conn_02x32_Odd_Even, J4 Conn_01x03_Pin, SW1 RESET, SW2 DEBUG, U1 74LS05, U10 74HC164, U11 74LS393, U12 22V10C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

Commit message: Re-added logo
Parts:
- D5: footprint Diode_THT:D_DO-27_P12.70mm_Horizontal -> Diode_THT:D_DO-41_SOD81_P7.62mm_Horizontal
Changed lines of the file:
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@@
       (effects (font (size 1.27 1.27)))
     )
-    (property "Footprint" "Diode_THT:D_DO-27_P12.70mm_Horizontal" (at 281.94 336.55 0)
+    (property "Footprint" "Diode_THT:D_DO-41_SOD81_P7.62mm_Horizontal" (at 281.94 336.55 0)
       (effects (font (size 1.27 1.27)) hide)
     )

Commit message: Fixed short trace to CC resistor
Parts:
- D5: value D_Schottky -> BAT85
Connections:
- net GND: now also U1.9
- no-connect marks 56 -> 57
Other:
- moved on the sheet: U1D
Changed lines of the file:
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@@
   (no_connect (at 62.23 139.7))
   (no_connect (at 194.31 205.74))
+  (no_connect (at 38.1 384.81))
   (no_connect (at 62.23 152.4))
   (no_connect (at 361.95 194.31))
@@
     (stroke (width 0) (type default))
   )
+  (wire (pts (xy 20.32 384.81) (xy 22.86 384.81))
+    (stroke (width 0) (type default))
+  )
   (bus (pts (xy 224.79 209.55) (xy 224.79 212.09))
     (stroke (width 0) (type default))
@@
     (stroke (width 0) (type default))
   )
+  (wire (pts (xy 20.32 384.81) (xy 20.32 387.35))
+    (stroke (width 0) (type default))
+  )
   (bus (pts (xy 321.31 40.64) (xy 321.31 43.18))
     (stroke (width 0) (type default))
@@
     )
   )
-  (symbol (lib_id "74xx:74LS05") (at 172.72 85.725 0) (unit 4)
+  (symbol (lib_id "74xx:74LS05") (at 30.48 384.81 0) (unit 4)
     (in_bom yes) (on_board yes) (dnp no) (fields_autoplaced)
-    (property "Reference" "U1" (at 172.72 77.597 0)
+    (property "Reference" "U1" (at 30.48 376.682 0)
       (effects (font (size 1.27 1.27)))
     )
-    (property "Value" "74LS05" (at 172.72 80.137 0)
+    (property "Value" "74LS05" (at 30.48 379.222 0)
       (effects (font (size 1.27 1.27)))
     )
-    (property "Footprint" "Package_DIP:DIP-14_W7.62mm_Socket" (at 172.72 85.725 0)
+    (property "Footprint" "Package_DIP:DIP-14_W7.62mm_Socket" (at 30.48 384.81 0)
       (effects (font (size 1.27 1.27)) hide)
     )
-    (property "Datasheet" "http://www.ti.com/lit/gpn/sn74LS05" (at 172.72 85.725 0)
+    (property "Datasheet" "http://www.ti.com/lit/gpn/sn74LS05" (at 30.48 384.81 0)
       (effects (font (size 1.27 1.27)) hide)
     )
@@
       (effects (font (size 1.27 1.27)))
     )
-    (property "Value" "D_Schottky" (at 281.6225 332.74 0)
+    (property "Value" "BAT85" (at 281.6225 332.74 0)
       (effects (font (size 1.27 1.27)))
     )
@@
         )
       )
+    )
+  )
+  (symbol (lib_id "power:GND") (at 20.32 387.35 0) (unit 1)
+    (in_bom yes) (on_board yes) (dnp no) (fields_autoplaced)
+    (property "Reference" "#PWR049" (at 20.32 393.7 0)
+      (effects (font (size 1.27 1.27)) hide)
+    )
+    (property "Value" "GND" (at 20.32 392.43 0)
+      (effects (font (size 1.27 1.27)))
+    )
+    (property "Footprint" "" (at 20.32 387.35 0)
+      (effects (font (size 1.27 1.27)) hide)
+    )
+    (property "Datasheet" "" (at 20.32 387.35 0)
+      (effects (font (size 1.27 1.27)) hide)
+    )
+    (pin "1")
+    (instances
+      (project "Sixty-n8k"
+        (path "/899701f7-f496-45c9-a35e-7f376afd1eaf"
+          (reference "#PWR049") (unit 1)
+        )
+      )
